File: Modules/BackPlane/PCB/BackPlane/BackPlane.kicad_pcb (KiCad board)
At the start: 2 copper layers, 80 x 34.3 mm, 5 parts

Commit message: Finished Sensor and Backplane boards
Parts:
- added G***: LOGO, IcaroFootprints:LogoGluon_25mm, F.Cu at (115.2, 92.4)
- added REF**: OSHW-Logo2_14.6x12mm_SilkScreen, Symbol:OSHW-Logo2_14.6x12mm_SilkScreen, F.Cu at (132.2, 93.5)
- added REF**: KiCad-Logo2_6mm_SilkScreen, Symbol:KiCad-Logo2_6mm_SilkScreen, F.Cu at (73.9, 91.5)
- added kibuzzard-67C807F8: G***, kibuzzard-67C807F8, F.Cu at (131.5, 55.9)
- added kibuzzard-67C807F8: G***, kibuzzard-67C807F8, B.Cu at (131.6, 55.9)
- added kibuzzard-67C80808: G***, kibuzzard-67C80808, F.Cu at (131.2, 73.7)
- added kibuzzard-67C80808: G***, kibuzzard-67C80808, F.Cu at (131.2, 58.4)
- added kibuzzard-67C80817: G***, kibuzzard-67C80817, F.Cu at (131.6, 61.0)
- added kibuzzard-67C80838: G***, kibuzzard-67C80838, F.Cu at (130.8, 63.5)
- added kibuzzard-67C80841: G***, kibuzzard-67C80841, F.Cu at (130.8, 66.0)
- added kibuzzard-67C80848: G***, kibuzzard-67C80848, F.Cu at (131.2, 68.6)
- added kibuzzard-67C80850: G***, kibuzzard-67C80850, F.Cu at (131.2, 71.4)
- added kibuzzard-67C80858: G***, kibuzzard-67C80858, F.Cu at (130.8, 76.2)
- added kibuzzard-67C80860: G***, kibuzzard-67C80860, F.Cu at (130.8, 78.7)
- added kibuzzard-67C80867: G***, kibuzzard-67C80867, F.Cu at (131.2, 81.3)
- added kibuzzard-67C8086E: G***, kibuzzard-67C8086E, F.Cu at (131.2, 83.8)
- added kibuzzard-67C808B4: G***, kibuzzard-67C808B4, B.Cu at (131.2, 58.4)
- added kibuzzard-67C808B4: G***, kibuzzard-67C808B4, B.Cu at (131.2, 73.7)
- added kibuzzard-67C808C7: G***, kibuzzard-67C808C7, B.Cu at (131.2, 61.0)
- added kibuzzard-67C808DE: G***, kibuzzard-67C808DE, B.Cu at (131.6, 63.5)
- added kibuzzard-67C808E6: G***, kibuzzard-67C808E6, B.Cu at (131.6, 66.0)
- added kibuzzard-67C808F2: G***, kibuzzard-67C808F2, B.Cu at (131.2, 68.6)
- added kibuzzard-67C808FD: G***, kibuzzard-67C808FD, B.Cu at (131.2, 71.1)
- added kibuzzard-67C80908: G***, kibuzzard-67C80908, B.Cu at (130.8, 76.2)
- added kibuzzard-67C8090F: G***, kibuzzard-67C8090F, B.Cu at (130.8, 78.7)
- added kibuzzard-67C80915: G***, kibuzzard-67C80915, B.Cu at (131.2, 81.3)
- added kibuzzard-67C8091B: G***, kibuzzard-67C8091B, B.Cu at (131.2, 83.8)
Connections:
- net /GND renamed GND
Routing:
- net GND: track 0.00 -> 307.1 mm
- net /BYPASS: track 0.00 -> 144.8 mm
- net /CS1: track 0.00 -> 94.3 mm
- net /SDA_0: track 0.00 -> 76.4 mm
- net /SCL_0: track 0.00 -> 76.4 mm
- net /IO2: track 0.00 -> 76.4 mm
- net /CS0: track 0.00 -> 76.4 mm
- net /SDA_1: track 0.00 -> 76.4 mm
- net /5V: track 0.00 -> 76.4 mm
- net /SCL_1: track 0.00 -> 76.4 mm
- net /IO0: track 0.00 -> 76.4 mm
- net /CS2: track 0.00 -> 76.4 mm
- net /MISO: track 0.00 -> 73.1 mm
- net /MOSI: track 0.00 -> 73.1 mm
- net /CS3: track 0.00 -> 73.0 mm
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Other:
- board size 80 x 34.3 mm -> 80 x 80 mm
- board text added: "Gracias!"
- board text added: "Proyecto Ícaro Backplane V1.0 by: @labgluon"
- board text added: "araba_st spuertes andygm_ zurano_ carlosbetdev gorn6_ david_wiki sergivv pipermind txusev enlopa blacai movich4 gordon_clark adiiran pulwef kerneltron victor_gomezzz alnaumiwebs dielek pintzio2 bark12 laboratoriocautin tuboniatofugaz t3l3mac0 rafaromevi hec100h diegomallo jotaperre jsochoa joseju_ch caramono_ maximoxx jositofotos crovodovod carbans"
