File: Modules/SensorBoard/PCB/SensorBoard/microcontroller.kicad_sch (KiCad schematic)
At the start: 0 parts

Commit message: sensor board basic components
Parts:
- added J5: PROG, Connector_PinHeader_2.54mm:PinHeader_1x04_P2.54mm_Vertical, symbol Connector_Generic:Conn_01x04
- added J7: Micro_SD_Card_Det1, IcaroFootprints:microSD-Receptacle-SelfEject, symbol Connector:Micro_SD_Card_Det1
- added U1: ESP32-WROOM-32D, RF_Module:ESP32-WROOM-32D, symbol RF_Module:ESP32-WROOM-32D
Connections:
- new net: U1.1 (GND), U1.15 (GND), U1.38 (GND), U1.39 (GND)

Commit message: Finished Supply board
Parts:
- removed J5: PROG, Connector_PinHeader_2.54mm:PinHeader_1x04_P2.54mm_Vertical, symbol Connector_Generic:Conn_01x04
- removed J7: Micro_SD_Card_Det1, IcaroFootprints:microSD-Receptacle-SelfEject, symbol Connector:Micro_SD_Card_Det1
- removed U1: ESP32-WROOM-32D, RF_Module:ESP32-WROOM-32D, symbol RF_Module:ESP32-WROOM-32D
- added C2: 100nF, Capacitor_SMD:C_0603_1608Metric_Pad1.08x0.95mm_HandSolder, symbol Device:C_Small
- added J6: Micro_SD_Card, IcaroFootprints:microSD-Receptacle-SelfEject, symbol Connector:Micro_SD_Card
- added J7: PROGRAMMING, Connector_PinHeader_2.54mm:PinHeader_1x04_P2.54mm_Vertical, symbol Connector_Generic:Conn_01x04
- added JP1: BOOT_SELECT, Connector_PinHeader_2.54mm:PinHeader_1x03_P2.54mm_Vertical, symbol Jumper:Jumper_3_Bridged12
- added R10, R11, R12, R20, R7, R8, R9: 10k, Resistor_SMD:R_0603_1608Metric_Pad0.98x0.95mm_HandSolder, symbol Device:R
- added U4: ESP32-WROOM-E, RF_Module:ESP32-WROOM-32UE, symbol Espressif:ESP32-WROOM-E
Connections:
- new net: C2.1, R7.1, U4.3 (EN/CHIP_PU)
- new net: JP1.2 (C), U4.25 (GPIO0/BOOT/ADC2_CH1)
- new net: J7.2 (Pin_2), U4.34 (U0RXD/GPIO3)
- new net: J7.3 (Pin_3), U4.35 (U0TXD/GPIO1)
- new net +3V3: J6.4 (VDD), J7.1 (Pin_1), JP1.1 (A), R10.2, R11.2, R12.2, R20.2, R7.2, R8.2, R9.2, U4.2 (3V3)
- new net GND: C2.2, J6.11 (SHIELD), J6.6 (VSS), J7.4 (Pin_4), JP1.3 (B), U4.1 (GND), U4.15 (GND), U4.38 (GND), U4.39 (GND_THERMAL)
- new net I2C_BME.SCL: U4.31 (GPIO19)
- new net I2C_BME.SDA: U4.30 (GPIO18)
- new net SD_CLK: J6.5 (CLK), U4.13 (MTMS/GPIO14/ADC2_CH6)
- new net SD_CMD: J6.3 (CMD), R10.1, U4.23 (MTDO/GPIO15/ADC2_CH3)
- new net SD_DATA0: J6.7 (DAT0), R11.1, U4.24 (ADC2_CH2/GPIO2)
- new net SD_DATA1: J6.8 (DAT1), R12.1, U4.26 (ADC2_CH0/GPIO4)
- new net SD_DATA2: J6.1 (DAT2), R8.1, U4.14 (MTDI/GPIO12/ADC2_CH5)
- new net SD_DATA3: J6.2 (DAT3/CD), R9.1, U4.16 (MTCK/GPIO13/ADC2_CH4)
- new net SPI_IMU.CS0: U4.12 (ADC2_CH7/GPIO27)
- new net SPI_IMU.MISO: U4.33 (GPIO21)
- new net SPI_IMU.MOSI: U4.36 (GPIO22)
- new net SPI_IMU.SCK: U4.37 (GPIO23)
- new net UART_GPS.RX: U4.27 (GPIO16)
- new net UART_GPS.TX: U4.28 (GPIO17)
- new net /CD_DETECT: J6.9 (CD), R20.1
- no-connect marks 0 -> 2
Other:
- note added: "Segun el ejemplo, hay que ponerlas de 10k https://github.com/espressif/esp-idf/blob/af805df3cb6117cc74f0875831fbab6446824453/examples/storage/sd_card/sdmmc/main/sd_card_example_main.c Linea 119"

Commit message: Enrutado de diseño de PT100 en la sensorboard
Parts:
- added D3: LED, LED_SMD:LED_0805_2012Metric_Pad1.15x1.40mm_HandSolder, symbol Device:LED
- added Q1: IRLM2502, Package_TO_SOT_SMD:SOT-23, symbol IcaroLib:IRLM2502
- added R25: 2k2, Resistor_SMD:R_0603_1608Metric_Pad0.98x0.95mm_HandSolder, symbol Device:R_Small
- added R26: 220, Resistor_SMD:R_0603_1608Metric_Pad0.98x0.95mm_HandSolder, symbol Device:R_Small
- added R27: 1Meg, Resistor_SMD:R_0603_1608Metric_Pad0.98x0.95mm_HandSolder, symbol Device:R_Small
- added U2: ~, IcaroFootprints:WheelSwitch, symbol IcaroLib:wheelSwitch
Connections:
- net I2C_BME.SCL is gone; now on net SPI_IMU.MISO: U4.31 (GPIO19)
- net I2C_BME.SDA is gone; now on net SPI_IMU.SCK: U4.30 (GPIO18)
- net /CD_DETECT is gone; now on net CD_DETECT: J6.9 (CD), R20.1
- net +3V3: now also R25.2
- net GND: now also Q1.2 (S), R27.1, U2.1 (COMMON)
- net SPI_IMU.CS0: now also U4.29 (GPIO5); no longer U4.12 (ADC2_CH7/GPIO27)
- net SPI_IMU.MISO: no longer U4.33 (GPIO21)
- net SPI_IMU.MOSI: now also U4.37 (GPIO23); no longer U4.36 (GPIO22)
- net SPI_IMU.SCK: no longer U4.37 (GPIO23)
- net I2C_EXT.SDA: now reaches U4.10 (DAC_1/ADC2_CH8/GPIO25)
- net I2C_EXT.SCL: now reaches U4.11 (DAC_2/ADC2_CH9/GPIO26)
- net at U4.25 (GPIO0/BOOT/ADC2_CH1): no longer JP1.2 (C)
- net UART_RX: now reaches J7.2 (Pin_2), U4.34 (U0RXD/GPIO3)
- net UART_TX: now reaches J7.3 (Pin_3), U4.35 (U0TXD/GPIO1)
- net CD_DETECT: now reaches U4.5 (SENSOR_VN/GPIO39/ADC1_CH3)
- net at U4.6 (GPIO34/ADC1_CH6): now also U2.2 (L)
- net at U4.7 (GPIO35/ADC1_CH7): now also U2.3 (Push)
- net at U4.8 (32K_XP/GPIO32/ADC1_CH4): now also U2.4 (R)
- new net: D3.2 (A), R25.1
- new net: D3.1 (K), Q1.3 (D)
- new net: Q1.1 (G), R26.1, R27.2
- new net I2C_INT.SCL: U4.36 (GPIO22)
- new net I2C_INT.SDA: U4.33 (GPIO21)
- new net LED_PIN: R26.2, U4.12 (ADC2_CH7/GPIO27)
Other:
- moved on the sheet: JP1

Commit message: Finished Sensor and Backplane boards
Connections:
- net at C2.1, R7.1, U4.3 (EN/CHIP_PU): now also U2.2 (L)
- net at U4.25 (GPIO0/BOOT/ADC2_CH1): now also JP1.2 (C)
- net at U4.6 (GPIO34/ADC1_CH6): no longer U2.2 (L)
- no-connect marks 2 -> 3
Other:
- moved on the sheet: J7, JP1
Changed lines of the file:
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@@
 	)
 	(no_connect
+		(at 132.08 86.36)
+	)
+	(no_connect
 		(at 128.27 93.98)
 	)
@@
 	(wire
 		(pts
-			(xy 95.25 73.66) (xy 95.25 74.93)
+			(xy 80.01 73.66) (xy 80.01 74.93)
 		)
 		(stroke
@@
 	(wire
 		(pts
-			(xy 92.71 73.66) (xy 95.25 73.66)
+			(xy 77.47 73.66) (xy 80.01 73.66)
 		)
 		(stroke
@@
 		)
 	)
+	(wire
+		(pts
+			(xy 107.95 54.61) (xy 119.38 54.61)
+		)
+		(stroke
+			(width 0)
+			(type default)
+		)
+	)
 	(bus
 		(pts
@@
 	(wire
 		(pts
-			(xy 52.07 86.36) (xy 52.07 87.63)
+			(xy 52.07 85.09) (xy 52.07 86.36)
 		)
 		(stroke
@@
 	(wire
 		(pts
-			(xy 92.71 68.58) (xy 132.08 68.58)
+			(xy 77.47 68.58) (xy 132.08 68.58)
+		)
+		(stroke
+			(width 0)
+			(type default)
+		)
+	)
+	(wire
+		(pts
+			(xy 107.95 85.09) (xy 107.95 54.61)
+		)
+		(stroke
+			(width 0)
+			(type default)
+		)
+	)
+	(wire
+		(pts
+			(xy 96.52 85.09) (xy 107.95 85.09)
 		)
 		(stroke
@@
 	(wire
 		(pts
-			(xy 92.71 66.04) (xy 100.33 66.04)
+			(xy 77.47 66.04) (xy 85.09 66.04)
 		)
 		(stroke
@@
 		)
 	)
-	(wire
-		(pts
-			(xy 111.76 86.36) (xy 132.08 86.36)
-		)
-		(stroke
-			(width 0)
-			(type default)
-		)
-	)
 	(bus
 		(pts
@@
 	(wire
 		(pts
-			(xy 52.07 71.12) (xy 52.07 73.66)
+			(xy 52.07 69.85) (xy 52.07 72.39)
 		)
 		(stroke
@@
 	(wire
 		(pts
-			(xy 92.71 71.12) (xy 132.08 71.12)
+			(xy 77.47 71.12) (xy 132.08 71.12)
 		)
 		(stroke
@@
 	(wire
 		(pts
-			(xy 100.33 66.04) (xy 100.33 64.77)
+			(xy 85.09 66.04) (xy 85.09 64.77)
 		)
 		(stroke
@@
 	(wire
 		(pts
-			(xy 111.76 85.09) (xy 111.76 86.36)
-		)
-		(stroke
-			(width 0)
-			(type default)
-		)
-	)
-	(wire
-		(pts
 			(xy 204.47 119.38) (xy 204.47 120.65)
 		)
@@
 	(wire
 		(pts
-			(xy 96.52 85.09) (xy 111.76 85.09)
-		)
-		(stroke
-			(width 0)
-			(type default)
-		)
-	)
-	(wire
-		(pts
 			(xy 246.38 143.51) (xy 248.92 143.51)
 		)
@@
 	)
 	(label "UART_TX"
-		(at 102.87 71.12 0)
+		(at 87.63 71.12 0)
 		(effects
 			(font
@@
 	)
 	(label "UART_RX"
-		(at 102.87 68.58 0)
+		(at 87.63 68.58 0)
 		(effects
 			(font
@@
 	(symbol
 		(lib_id "power:GND")
-		(at 52.07 87.63 0)
+		(at 52.07 86.36 0)
 		(unit 1)
 		(exclude_from_sim no)
@@
 		(dnp no)
 		(property "Reference" "#PWR015"
-			(at 52.07 93.98 0)
+			(at 52.07 92.71 0)
 			(effects
 				(font
@@
 		)
 		(property "Value" "GND"
-			(at 46.355 88.9 0)
+			(at 46.355 87.63 0)
 			(effects
 				(font
@@
 		)
 		(property "Footprint" ""
-			(at 52.07 87.63 0)
+			(at 52.07 86.36 0)
 			(effects
 				(font
@@
 		)
 		(property "Datasheet" ""
-			(at 52.07 87.63 0)
+			(at 52.07 86.36 0)
 			(effects
 				(font
@@
 		)
 		(property "Description" ""
-			(at 52.07 87.63 0)
+			(at 52.07 86.36 0)
 			(effects
 				(font
@@
 	(symbol
 		(lib_id "power:+3V3")
-		(at 52.07 71.12 0)
+		(at 52.07 69.85 0)
 		(unit 1)
 		(exclude_from_sim no)
@@
 		(fields_autoplaced yes)
 		(property "Reference" "#PWR014"
-			(at 52.07 74.93 0)
+			(at 52.07 73.66 0)
 			(effects
 				(font
@@
 		)
 		(property "Value" "+3V3"
-			(at 50.673 70.2838 0)
+			(at 50.673 69.0138 0)
 			(effects
 				(font
@@
 		)
 		(property "Footprint" ""
-			(at 52.07 71.12 0)
+			(at 52.07 69.85 0)
 			(effects
 				(font
@@
 		)
 		(property "Datasheet" ""
-			(at 52.07 71.12 0)
+			(at 52.07 69.85 0)
 			(effects
 				(font
@@
 		)
 		(property "Description" ""
-			(at 52.07 71.12 0)
+			(at 52.07 69.85 0)
 			(effects
 				(font
@@
 	(symbol
 		(lib_id "power:GND")
-		(at 95.25 74.93 0)
+		(at 80.01 74.93 0)
 		(unit 1)
 		(exclude_from_sim no)
@@
 		(dnp no)
 		(property "Reference" "#PWR09"
-			(at 95.25 81.28 0)
+			(at 80.01 81.28 0)
 			(effects
 				(font
@@
 		)
 		(property "Value" "GND"
-			(at 89.535 76.2 0)
+			(at 74.295 76.2 0)
 			(effects
 				(font
@@
 		)
 		(property "Footprint" ""
-			(at 95.25 74.93 0)
+			(at 80.01 74.93 0)
 			(effects
 				(font
@@
 		)
 		(property "Datasheet" ""
-			(at 95.25 74.93 0)
+			(at 80.01 74.93 0)
 			(effects
 				(font
@@
 		)
 		(property "Description" ""
-			(at 95.25 74.93 0)
+			(at 80.01 74.93 0)
 			(effects
 				(font
@@
 	(symbol
 		(lib_id "power:+3V3")
-		(at 100.33 64.77 0)
+		(at 85.09 64.77 0)
 		(unit 1)
 		(exclude_from_sim no)
@@
 		(fields_autoplaced yes)
 		(property "Reference" "#PWR08"
-			(at 100.33 68.58 0)
+			(at 85.09 68.58 0)
 			(effects
 				(font
@@
 		)
 		(property "Value" "+3V3"
-			(at 100.33 61.1942 0)
+			(at 85.09 61.1942 0)
 			(effects
 				(font
@@
 		)
 		(property "Footprint" ""
-			(at 100.33 64.77 0)
+			(at 85.09 64.77 0)
 			(effects
 				(font
@@
 		)
 		(property "Datasheet" ""
-			(at 100.33 64.77 0)
+			(at 85.09 64.77 0)
 			(effects
 				(font
@@
 		)
 		(property "Description" ""
-			(at 100.33 64.77 0)
+			(at 85.09 64.77 0)
 			(effects
 				(font
@@
 	(symbol
 		(lib_id "Jumper:Jumper_3_Bridged12")
-		(at 52.07 80.01 90)
+		(at 52.07 78.74 90)
 		(mirror x)
 		(unit 1)
@@
 		(dnp no)
 		(property "Reference" "JP1"
-			(at 48.26 78.74 90)
+			(at 48.26 77.47 90)
 			(effects
 				(font
@@
 		)
 		(property "Value" "BOOT_SELECT"
-			(at 43.815 80.645 90)
+			(at 43.815 79.375 90)
 			(effects
 				(font
@@
 		)
 		(property "Footprint" "Connector_PinHeader_2.54mm:PinHeader_1x03_P2.54mm_Vertical"
-			(at 52.07 80.01 0)
+			(at 52.07 78.74 0)
 			(effects
 				(font
@@
 		)
 		(property "Datasheet" "~"
-			(at 52.07 80.01 0)
+			(at 52.07 78.74 0)
 			(effects
 				(font
@@
 		)
 		(property "Description" ""
-			(at 52.07 80.01 0)
+			(at 52.07 78.74 0)
 			(effects
 				(font
@@
 	(symbol
 		(lib_id "Connector_Generic:Conn_01x04")
-		(at 87.63 68.58 0)
+		(at 72.39 68.58 0)
 		(mirror y)
 		(unit 1)
@@
 		(fields_autoplaced yes)
 		(property "Reference" "J7"
-			(at 85.598 69.0153 0)
+			(at 70.358 69.0153 0)
 			(effects
 				(font
@@
 		)
 		(property "Value" "PROGRAMMING"
-			(at 85.598 71.5522 0)
+			(at 70.358 71.5522 0)
 			(effects
 				(font
@@
 		)
 		(property "Footprint" "Connector_PinHeader_2.54mm:PinHeader_1x04_P2.54mm_Vertical"
-			(at 87.63 68.58 0)
+			(at 72.39 68.58 0)
 			(effects
 				(font
@@
 		)
 		(property "Datasheet" "~"
-			(at 87.63 68.58 0)
+			(at 72.39 68.58 0)
 			(effects
 				(font
@@
 		)
 		(property "Description" ""
-			(at 87.63 68.58 0)
+			(at 72.39 68.58 0)
 			(effects
 				(font
